File: right/ortho_right.kicad_pcb (KiCad board)
At the start: 2 copper layers, 189.2 x 146.1 mm, 75 parts, among them J1 AudioJack4, J10 Conn_01x01, J11 Conn_01x01, J12 Conn_01x01, J13 Conn_01x01, J2 Conn_01x01, J3 Conn_01x01, J4 Conn_01x01, J5 Conn_01x01, J6 Conn_01x01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

Commit message: Kicad 6 migration; other fixes
Other:
- net class Default removed
