File: left/LEDs.kicad_sch (KiCad schematic)
At the start: 40 parts, among them J18 Conn_01x01, J19 Conn_01x01, J20 Conn_01x01, J21 Conn_01x01, K11 KEYSW_RGB, K12 KEYSW_RGB, K13 KEYSW_RGB, K14 KEYSW_RGB, K15 KEYSW_RGB, K16 KEYSW_RGB, K21 KEYSW_RGB, K22 KEYSW_RGB, K23 KEYSW_RGB, K24 KEYSW_RGB, K25 KEYSW_RGB, K26 KEYSW_RGB, K31 KEYSW_RGB, K32 KEYSW_RGB, K33 KEYSW_RGB, K34 KEYSW_RGB, K35 KEYSW_RGB, K36 KEYSW_RGB, K41 KEYSW_RGB, K42 KEYSW_RGB, K43 KEYSW_RGB, K44 KEYSW_RGB, K45 KEYSW_RGB, K46 KEYSW_RGB, K51 KEYSW_RGB, K52 KEYSW_RGB, K53 KEYSW_RGB, K54 KEYSW_RGB, K55 KEYSW_RGB, K56 KEYSW_RGB, K61 KEYSW_RGB, K62 KEYSW_RGB, K63 KEYSW_RGB, K64 KEYSW_RGB, K65 KEYSW_RGB, K66 KEYSW_RGB

Commit message: Broke out keys into individual components so that the BOM and pick and place are easier to generate.
Parts:
- removed J18, J19, J20, J21: Conn_01x01, TestPoint:TestPoint_Pad_D1.5mm, symbol Connector_Generic:Conn_01x01
- removed K11, K21, K31, K41, K51: KEYSW_RGB, vladkvit_keyb:Hybrid_PCB_150H_hotswap_diode_RGB_rot, symbol vladkvit_keyb:KEYSW_RGB
- removed K12, K13, K14, K15, K16, K22, K23, K24, K25, K26, K32, K33, K34, K35, K36, K42, K43, K44, K45, K46, K52, K53, K54, K55, K56: KEYSW_RGB, vladkvit_keyb:Hybrid_PCB_100H_hotswap_diode_RGB_rot, symbol vladkvit_keyb:KEYSW_RGB
- removed K61, K62, K63, K64: KEYSW_RGB, vladkvit_keyb:Hybrid_PCB_125H_hotswap_diode_RGB_rot, symbol vladkvit_keyb:KEYSW_RGB
- removed K65, K66: KEYSW_RGB, vladkvit_keyb:Hybrid_PCB_200H_hotswap_diode_RGB, symbol vladkvit_keyb:KEYSW_RGB
