File: left/hierarchical_keys.kicad_sch (KiCad schematic)
At the start: 3 parts, among them K34 KEYSW

Commit message: Kicad 9 upgrade.
Parts:
- D12: renamed from D34; LCSC (none) -> C6958246
- D121: renamed from D341; LCSC (none) -> C77978
- K12: renamed from K34; LCSC (none) -> C5156480
Changed lines of the file:
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@@
 (kicad_sch
-	(version 20231120)
+	(version 20250114)
 	(generator "eeschema")
-	(generator_version "8.0")
+	(generator_version "9.0")
 	(paper "A4")
 	(hierarchical_label "RGB_R"
 		(shape input)
 		(at 161.29 113.03 180)
-		(fields_autoplaced yes)
 		(effects
 			(font
@@
 		(shape input)
 		(at 171.45 118.11 0)
-		(fields_autoplaced yes)
 		(effects
 			(font
@@
 		(shape input)
 		(at 161.29 123.19 180)
-		(fields_autoplaced yes)
 		(effects
 			(font
@@
 		(shape input)
 		(at 124.46 110.49 180)
-		(fields_autoplaced yes)
 		(effects
 			(font
@@
 		(shape input)
 		(at 134.62 118.11 270)
-		(fields_autoplaced yes)
 		(effects
 			(font
@@
 		(shape input)
 		(at 161.29 118.11 180)
-		(fields_autoplaced yes)
 		(effects
 			(font
@@
 		(dnp no)
 		(fields_autoplaced yes)
-		(property "Reference" "D34"
+		(property "Reference" "D12"
 			(at 166.37 104.14 0)
 			(effects
@@
 			)
 		)
-		(property "Description" "RGB LED, anode/red/green/blue"
+		(property "Description" "RGB LED, anode/red/green/blue, Any of: QBLP677R-RGB  T36K3BGR-05D000121U1930  IN-P32TRRRGB"
+			(at 166.37 118.11 0)
+			(effects
+				(font
+					(size 1.27 1.27)
+				)
+				(hide yes)
+			)
+		)
+		(property "LCSC" "C6958246"
 			(at 166.37 118.11 0)
 			(effects
@@
 					(unit 1)
 				)
-				(path "/0217dfc4-fc13-4699-99ad-d9948522648e/00000000-0000-0000-0000-00005f15430e/19c1d365-e8c3-487b-8bb3-33a31c7800ff"
-					(reference "D65")
-					(unit 1)
-				)
-				(path "/0217dfc4-fc13-4699-99ad-d9948522648e/00000000-0000-0000-0000-00005f15430e/1e53d279-95db-481a-a48c-a1712c6ef226"
-					(reference "D63")
-					(unit 1)
-				)
 				(path "/0217dfc4-fc13-4699-99ad-d9948522648e/00000000-0000-0000-0000-00005f15430e/1eec75c9-c11d-4544-bcdb-e911bfda2032"
 					(reference "D53")
@@
 					(unit 1)
 				)
-				(path "/0217dfc4-fc13-4699-99ad-d9948522648e/00000000-0000-0000-0000-00005f15430e/4008de6f-ce59-4bfc-bb4a-9cce8a715cca"
-					(reference "D66")
-					(unit 1)
-				)
 				(path "/0217dfc4-fc13-4699-99ad-d9948522648e/00000000-0000-0000-0000-00005f15430e/434d555c-4a4e-4b25-b5a5-baded7f12a85"
 					(reference "D33")
@@
 					(unit 1)
 				)
-				(path "/0217dfc4-fc13-4699-99ad-d9948522648e/00000000-0000-0000-0000-00005f15430e/7a67f58e-a4de-4fd2-a981-d4ac0c2905fb"
-					(reference "D62")
-					(unit 1)
-				)
 				(path "/0217dfc4-fc13-4699-99ad-d9948522648e/00000000-0000-0000-0000-00005f15430e/7d7a0dc2-94e3-449c-9778-63ad4ccc4129"
 					(reference "D15")
@@
 					(unit 1)
 				)
-				(path "/0217dfc4-fc13-4699-99ad-d9948522648e/00000000-0000-0000-0000-00005f15430e/a81301bf-ba37-4b8b-9ec9-19ddb291a549"
-					(reference "D64")
-					(unit 1)
-				)
 				(path "/0217dfc4-fc13-4699-99ad-d9948522648e/00000000-0000-0000-0000-00005f15430e/ae49d6cc-07ee-49a8-ae09-548872a8ca60"
 					(reference "D32")
@@
 				(path "/0217dfc4-fc13-4699-99ad-d9948522648e/00000000-0000-0000-0000-00005f15430e/c56680ba-355f-4c31-96ba-a37dd99fe7fa"
 					(reference "D36")
-					(unit 1)
-				)
-				(path "/0217dfc4-fc13-4699-99ad-d9948522648e/00000000-0000-0000-0000-00005f15430e/d1e0a952-b6a6-4bf6-93c1-011396209d0f"
-					(reference "D61")
 					(unit 1)
 				)
@@
 		(on_board yes)
 		(dnp no)
-		(property "Reference" "K34"
+		(property "Reference" "K12"
 			(at 128.27 104.5718 0)
 			(effects
@@
 			)
 		)
-		(property "Description" "Push button switch, generic, two pins"
+		(property "Description" "Hot swap socket, CPG151101S11 or similar, C5156480 or C5184526"
+			(at 129.54 110.49 0)
+			(effects
+				(font
+					(size 1.27 1.27)
+				)
+				(hide yes)
+			)
+		)
+		(property "LCSC" "C5156480"
 			(at 129.54 110.49 0)
 			(effects
@@
 					(unit 1)
 				)
-				(path "/0217dfc4-fc13-4699-99ad-d9948522648e/00000000-0000-0000-0000-00005f15430e/19c1d365-e8c3-487b-8bb3-33a31c7800ff"
-					(reference "K65")
-					(unit 1)
-				)
-				(path "/0217dfc4-fc13-4699-99ad-d9948522648e/00000000-0000-0000-0000-00005f15430e/1e53d279-95db-481a-a48c-a1712c6ef226"
-					(reference "K63")
-					(unit 1)
-				)
 				(path "/0217dfc4-fc13-4699-99ad-d9948522648e/00000000-0000-0000-0000-00005f15430e/1eec75c9-c11d-4544-bcdb-e911bfda2032"
 					(reference "K53")
@@
 					(unit 1)
 				)
-				(path "/0217dfc4-fc13-4699-99ad-d9948522648e/00000000-0000-0000-0000-00005f15430e/4008de6f-ce59-4bfc-bb4a-9cce8a715cca"
-					(reference "K66")
-					(unit 1)
-				)
 				(path "/0217dfc4-fc13-4699-99ad-d9948522648e/00000000-0000-0000-0000-00005f15430e/434d555c-4a4e-4b25-b5a5-baded7f12a85"
 					(reference "K33")
@@
 					(unit 1)
 				)
-				(path "/0217dfc4-fc13-4699-99ad-d9948522648e/00000000-0000-0000-0000-00005f15430e/7a67f58e-a4de-4fd2-a981-d4ac0c2905fb"
-					(reference "K62")
-					(unit 1)
-				)
 				(path "/0217dfc4-fc13-4699-99ad-d9948522648e/00000000-0000-0000-0000-00005f15430e/7d7a0dc2-94e3-449c-9778-63ad4ccc4129"
 					(reference "K15")
@@
 					(unit 1)
 				)
-				(path "/0217dfc4-fc13-4699-99ad-d9948522648e/00000000-0000-0000-0000-00005f15430e/a81301bf-ba37-4b8b-9ec9-19ddb291a549"
-					(reference "K64")
-					(unit 1)
-				)
 				(path "/0217dfc4-fc13-4699-99ad-d9948522648e/00000000-0000-0000-0000-00005f15430e/ae49d6cc-07ee-49a8-ae09-548872a8ca60"
 					(reference "K32")
@@
 				(path "/0217dfc4-fc13-4699-99ad-d9948522648e/00000000-0000-0000-0000-00005f15430e/c56680ba-355f-4c31-96ba-a37dd99fe7fa"
 					(reference "K36")
-					(unit 1)
-				)
-				(path "/0217dfc4-fc13-4699-99ad-d9948522648e/00000000-0000-0000-0000-00005f15430e/d1e0a952-b6a6-4bf6-93c1-011396209d0f"
-					(reference "K61")
 					(unit 1)
 				)
@@
 		(dnp no)
 		(fields_autoplaced yes)
-		(property "Reference" "D341"
+		(property "Reference" "D121"
 			(at 137.16 113.0299 90)
 			(effects
@@
 			)
 		)
-		(property "Description" "Diode"
+		(property "Description" "Diode, Any 1N4148"
 			(at 134.62 114.3 0)
 			(effects
@@
 		)
 		(property "Sim.Pins" "1=K 2=A"
+			(at 134.62 114.3 0)
+			(effects
+				(font
+					(size 1.27 1.27)
+				)
+				(hide yes)
+			)
+		)
+		(property "LCSC" "C77978"
 			(at 134.62 114.3 0)
 			(effects
@@
 					(unit 1)
 				)
-				(path "/0217dfc4-fc13-4699-99ad-d9948522648e/00000000-0000-0000-0000-00005f15430e/19c1d365-e8c3-487b-8bb3-33a31c7800ff"
-					(reference "D651")
-					(unit 1)
-				)
-				(path "/0217dfc4-fc13-4699-99ad-d9948522648e/00000000-0000-0000-0000-00005f15430e/1e53d279-95db-481a-a48c-a1712c6ef226"
-					(reference "D631")
-					(unit 1)
-				)
 				(path "/0217dfc4-fc13-4699-99ad-d9948522648e/00000000-0000-0000-0000-00005f15430e/1eec75c9-c11d-4544-bcdb-e911bfda2032"
 					(reference "D531")
@@
 					(unit 1)
 				)
-				(path "/0217dfc4-fc13-4699-99ad-d9948522648e/00000000-0000-0000-0000-00005f15430e/4008de6f-ce59-4bfc-bb4a-9cce8a715cca"
-					(reference "D661")
-					(unit 1)
-				)
 				(path "/0217dfc4-fc13-4699-99ad-d9948522648e/00000000-0000-0000-0000-00005f15430e/434d555c-4a4e-4b25-b5a5-baded7f12a85"
 					(reference "D331")
@@
 					(unit 1)
 				)
-				(path "/0217dfc4-fc13-4699-99ad-d9948522648e/00000000-0000-0000-0000-00005f15430e/7a67f58e-a4de-4fd2-a981-d4ac0c2905fb"
-					(reference "D621")
-					(unit 1)
-				)
 				(path "/0217dfc4-fc13-4699-99ad-d9948522648e/00000000-0000-0000-0000-00005f15430e/7d7a0dc2-94e3-449c-9778-63ad4ccc4129"
 					(reference "D151")
@@
 					(unit 1)
 				)
-				(path "/0217dfc4-fc13-4699-99ad-d9948522648e/00000000-0000-0000-0000-00005f15430e/a81301bf-ba37-4b8b-9ec9-19ddb291a549"
-					(reference "D641")
-					(unit 1)
-				)
 				(path "/0217dfc4-fc13-4699-99ad-d9948522648e/00000000-0000-0000-0000-00005f15430e/ae49d6cc-07ee-49a8-ae09-548872a8ca60"
 					(reference "D321")
@@
 					(unit 1)
 				)
-				(path "/0217dfc4-fc13-4699-99ad-d9948522648e/00000000-0000-0000-0000-00005f15430e/d1e0a952-b6a6-4bf6-93c1-011396209d0f"
-					(reference "D611")
-					(unit 1)
-				)
