File: left/hierarchical_keys_150.kicad_sch (KiCad schematic)
At the start: 3 parts, among them K11 KEYSW

Commit message: Kicad 9 upgrade.
Parts:
- D11: LCSC (none) -> C6958246
- D111: LCSC (none) -> C77978
- K11: LCSC (none) -> C5156480
Changed lines of the file:
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@@
 (kicad_sch
-	(version 20231120)
+	(version 20250114)
 	(generator "eeschema")
-	(generator_version "8.0")
+	(generator_version "9.0")
 	(paper "A4")
 	(hierarchical_label "RGB_G"
 		(shape input)
 		(at 161.29 118.11 180)
-		(fields_autoplaced yes)
 		(effects
 			(font
@@
 		(shape input)
 		(at 161.29 113.03 180)
-		(fields_autoplaced yes)
 		(effects
 			(font
@@
 		(shape input)
 		(at 161.29 123.19 180)
-		(fields_autoplaced yes)
 		(effects
 			(font
@@
 		(shape input)
 		(at 134.62 118.11 270)
-		(fields_autoplaced yes)
 		(effects
 			(font
@@
 		(shape input)
 		(at 124.46 110.49 180)
-		(fields_autoplaced yes)
 		(effects
 			(font
@@
 		(shape input)
 		(at 171.45 118.11 0)
-		(fields_autoplaced yes)
 		(effects
 			(font
@@
 			)
 		)
-		(property "Description" "Diode"
+		(property "Description" "Diode, Any 1N4148"
 			(at 134.62 114.3 0)
 			(effects
@@
 		)
 		(property "Sim.Pins" "1=K 2=A"
+			(at 134.62 114.3 0)
+			(effects
+				(font
+					(size 1.27 1.27)
+				)
+				(hide yes)
+			)
+		)
+		(property "LCSC" "C77978"
 			(at 134.62 114.3 0)
 			(effects
@@
 			)
 		)
-		(property "Description" "Push button switch, generic, two pins"
+		(property "Description" "Hot swap socket, CPG151101S11 or similar, C5156480 or C5184526"
+			(at 129.54 110.49 0)
+			(effects
+				(font
+					(size 1.27 1.27)
+				)
+				(hide yes)
+			)
+		)
+		(property "LCSC" "C5156480"
 			(at 129.54 110.49 0)
 			(effects
@@
 			)
 		)
-		(property "Description" "RGB LED, anode/red/green/blue"
+		(property "Description" "RGB LED, anode/red/green/blue, Any of: QBLP677R-RGB  T36K3BGR-05D000121U1930  IN-P32TRRRGB"
 			(at 166.37 118.11 0)
 			(effects
+				(font
+					(size 1.27 1.27)
+				)
+				(hide yes)
+			)
+		)
+		(property "LCSC" "C6958246"
+			(at 166.37 118.11 0)
+			(effects
