File: left/hierarchical_keys_200.kicad_sch (KiCad schematic)
At the start: 3 parts, among them K31 KEYSW

Commit message: Kicad 9 upgrade.
Parts:
- D65: renamed from D31; LCSC (none) -> C6958246
- D651: renamed from D311; LCSC (none) -> C77978
- K65: renamed from K31; LCSC (none) -> C5156480
Changed lines of the file:
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@@
 (kicad_sch
-	(version 20231120)
+	(version 20250114)
 	(generator "eeschema")
-	(generator_version "8.0")
+	(generator_version "9.0")
 	(paper "A4")
 	(hierarchical_label "RGB_B"
 		(shape input)
 		(at 161.29 123.19 180)
-		(fields_autoplaced yes)
 		(effects
 			(font
@@
 		(shape input)
 		(at 134.62 118.11 270)
-		(fields_autoplaced yes)
 		(effects
 			(font
@@
 		(shape input)
 		(at 161.29 118.11 180)
-		(fields_autoplaced yes)
 		(effects
 			(font
@@
 		(shape input)
 		(at 161.29 113.03 180)
-		(fields_autoplaced yes)
 		(effects
 			(font
@@
 		(shape input)
 		(at 171.45 118.11 0)
-		(fields_autoplaced yes)
 		(effects
 			(font
@@
 		(shape input)
 		(at 124.46 110.49 180)
-		(fields_autoplaced yes)
 		(effects
 			(font
@@
 		(dnp no)
 		(fields_autoplaced yes)
-		(property "Reference" "D31"
+		(property "Reference" "D65"
 			(at 166.37 104.14 0)
 			(effects
@@
 			)
 		)
-		(property "Description" "RGB LED, anode/red/green/blue"
+		(property "Description" "RGB LED, anode/red/green/blue, Any of: QBLP677R-RGB  T36K3BGR-05D000121U1930  IN-P32TRRRGB"
+			(at 166.37 118.11 0)
+			(effects
+				(font
+					(size 1.27 1.27)
+				)
+				(hide yes)
+			)
+		)
+		(property "LCSC" "C6958246"
 			(at 166.37 118.11 0)
 			(effects
@@
 		(instances
 			(project "ortho_half"
-				(path "/0217dfc4-fc13-4699-99ad-d9948522648e/00000000-0000-0000-0000-00005f15430e/16161786-71b3-42fd-a9ab-f0dbf2dce39d"
-					(reference "D31")
-					(unit 1)
-				)
 				(path "/0217dfc4-fc13-4699-99ad-d9948522648e/00000000-0000-0000-0000-00005f15430e/19c1d365-e8c3-487b-8bb3-33a31c7800ff"
 					(reference "D65")
 					(unit 1)
 				)
-				(path "/0217dfc4-fc13-4699-99ad-d9948522648e/00000000-0000-0000-0000-00005f15430e/36e2917c-9df6-4d49-a877-495fe5c36a3e"
-					(reference "D51")
-					(unit 1)
-				)
 				(path "/0217dfc4-fc13-4699-99ad-d9948522648e/00000000-0000-0000-0000-00005f15430e/4008de6f-ce59-4bfc-bb4a-9cce8a715cca"
 					(reference "D66")
-					(unit 1)
-				)
-				(path "/0217dfc4-fc13-4699-99ad-d9948522648e/00000000-0000-0000-0000-00005f15430e/6a7a0925-9918-4e5b-9b45-c1c8e836020b"
-					(reference "D41")
-					(unit 1)
-				)
-				(path "/0217dfc4-fc13-4699-99ad-d9948522648e/00000000-0000-0000-0000-00005f15430e/a228be83-5b7e-47a6-8b4a-8f4c38a75eb0"
-					(reference "D11")
-					(unit 1)
-				)
-				(path "/0217dfc4-fc13-4699-99ad-d9948522648e/00000000-0000-0000-0000-00005f15430e/b98c62e9-36b0-45ff-b13a-56319ad05470"
-					(reference "D21")
 					(unit 1)
 				)
@@
 		(on_board yes)
 		(dnp no)
-		(property "Reference" "K31"
+		(property "Reference" "K65"
 			(at 128.27 104.5718 0)
 			(effects
@@
 			)
 		)
-		(property "Description" "Push button switch, generic, two pins"
+		(property "Description" "Hot swap socket, CPG151101S11 or similar, C5156480 or C5184526"
+			(at 129.54 110.49 0)
+			(effects
+				(font
+					(size 1.27 1.27)
+				)
+				(hide yes)
+			)
+		)
+		(property "LCSC" "C5156480"
 			(at 129.54 110.49 0)
 			(effects
@@
 		(instances
 			(project "ortho_half"
-				(path "/0217dfc4-fc13-4699-99ad-d9948522648e/00000000-0000-0000-0000-00005f15430e/16161786-71b3-42fd-a9ab-f0dbf2dce39d"
-					(reference "K31")
-					(unit 1)
-				)
 				(path "/0217dfc4-fc13-4699-99ad-d9948522648e/00000000-0000-0000-0000-00005f15430e/19c1d365-e8c3-487b-8bb3-33a31c7800ff"
 					(reference "K65")
 					(unit 1)
 				)
-				(path "/0217dfc4-fc13-4699-99ad-d9948522648e/00000000-0000-0000-0000-00005f15430e/36e2917c-9df6-4d49-a877-495fe5c36a3e"
-					(reference "K51")
-					(unit 1)
-				)
 				(path "/0217dfc4-fc13-4699-99ad-d9948522648e/00000000-0000-0000-0000-00005f15430e/4008de6f-ce59-4bfc-bb4a-9cce8a715cca"
 					(reference "K66")
-					(unit 1)
-				)
-				(path "/0217dfc4-fc13-4699-99ad-d9948522648e/00000000-0000-0000-0000-00005f15430e/6a7a0925-9918-4e5b-9b45-c1c8e836020b"
-					(reference "K41")
-					(unit 1)
-				)
-				(path "/0217dfc4-fc13-4699-99ad-d9948522648e/00000000-0000-0000-0000-00005f15430e/a228be83-5b7e-47a6-8b4a-8f4c38a75eb0"
-					(reference "K11")
-					(unit 1)
-				)
-				(path "/0217dfc4-fc13-4699-99ad-d9948522648e/00000000-0000-0000-0000-00005f15430e/b98c62e9-36b0-45ff-b13a-56319ad05470"
-					(reference "K21")
 					(unit 1)
 				)
@@
 		(dnp no)
 		(fields_autoplaced yes)
-		(property "Reference" "D311"
+		(property "Reference" "D651"
 			(at 137.16 113.0299 90)
 			(effects
@@
 			)
 		)
-		(property "Description" "Diode"
+		(property "Description" "Diode, Any 1N4148"
 			(at 134.62 114.3 0)
 			(effects
@@
 		)
 		(property "Sim.Pins" "1=K 2=A"
+			(at 134.62 114.3 0)
+			(effects
+				(font
+					(size 1.27 1.27)
+				)
+				(hide yes)
+			)
+		)
+		(property "LCSC" "C77978"
 			(at 134.62 114.3 0)
 			(effects
@@
 		(instances
 			(project "ortho_half"
-				(path "/0217dfc4-fc13-4699-99ad-d9948522648e/00000000-0000-0000-0000-00005f15430e/16161786-71b3-42fd-a9ab-f0dbf2dce39d"
-					(reference "D311")
-					(unit 1)
-				)
 				(path "/0217dfc4-fc13-4699-99ad-d9948522648e/00000000-0000-0000-0000-00005f15430e/19c1d365-e8c3-487b-8bb3-33a31c7800ff"
 					(reference "D651")
 					(unit 1)
 				)
-				(path "/0217dfc4-fc13-4699-99ad-d9948522648e/00000000-0000-0000-0000-00005f15430e/36e2917c-9df6-4d49-a877-495fe5c36a3e"
-					(reference "D511")
-					(unit 1)
-				)
 				(path "/0217dfc4-fc13-4699-99ad-d9948522648e/00000000-0000-0000-0000-00005f15430e/4008de6f-ce59-4bfc-bb4a-9cce8a715cca"
 					(reference "D661")
 					(unit 1)
 				)
-				(path "/0217dfc4-fc13-4699-99ad-d9948522648e/00000000-0000-0000-0000-00005f15430e/6a7a0925-9918-4e5b-9b45-c1c8e836020b"
-					(reference "D411")
-					(unit 1)
-				)
-				(path "/0217dfc4-fc13-4699-99ad-d9948522648e/00000000-0000-0000-0000-00005f15430e/a228be83-5b7e-47a6-8b4a-8f4c38a75eb0"
-					(reference "D111")
-					(unit 1)
-				)
-				(path "/0217dfc4-fc13-4699-99ad-d9948522648e/00000000-0000-0000-0000-00005f15430e/b98c62e9-36b0-45ff-b13a-56319ad05470"
-					(reference "D211")
-					(unit 1)
-				)
